File: schematics.kicad_sch (KiCad schematic)
At the start: 7 parts, among them J1 iBUS Sensor, J2 iBUS Servo, J3 BATT, J4 OLED, J5 TPS61023, SW2 Switch, U1 XIAO-ESP32-C6-SMD

Commit message: readme
Connections:
- net D_IN: now also U1.8 (D7); no longer U1.1 (D0)
- net D_OUT: now also U1.7 (D6); no longer U1.2 (D1)
Changed lines of the file:
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@@
+	(wire
+		(pts
+			(xy 99.06 81.28) (xy 105.41 81.28)
+		)
+		(stroke
+			(width 0)
+			(type default)
+		)
+	)
 	(wire
 		(pts
@@
 	(wire
 		(pts
+			(xy 151.13 81.28) (xy 154.94 81.28)
+		)
+		(stroke
+			(width 0)
+			(type default)
+		)
+	)
+	(wire
+		(pts
 			(xy 151.13 62.23) (xy 153.67 62.23)
 		)
@@
 	(wire
 		(pts
-			(xy 99.06 62.23) (xy 105.41 62.23)
-		)
-		(stroke
-			(width 0)
-			(type default)
-		)
-	)
-	(wire
-		(pts
 			(xy 124.46 87.63) (xy 124.46 91.44)
 		)
@@
 		(pts
 			(xy 99.06 73.66) (xy 105.41 73.66)
-		)
-		(stroke
-			(width 0)
-			(type default)
-		)
-	)
-	(wire
-		(pts
-			(xy 99.06 58.42) (xy 105.41 58.42)
 		)
 		(stroke
@@
 		)
 	)
-	(label "D_IN"
-		(at 99.06 58.42 0)
-		(effects
-			(font
-				(size 1.27 1.27)
-			)
-			(justify left bottom)
-		)
-	)
 	(label "SCK"
 		(at 99.06 77.47 0)
@@
 		)
 	)
-	(label "D_OUT"
-		(at 99.06 62.23 0)
-		(effects
-			(font
-				(size 1.27 1.27)
-			)
-			(justify left bottom)
-		)
-	)
 	(label "SDA"
 		(at 99.06 73.66 0)
@@
 		)
 	)
+	(label "D_IN"
+		(at 154.94 81.28 0)
+		(effects
+			(font
+				(size 1.27 1.27)
+			)
+			(justify left bottom)
+		)
+	)
+	(label "D_OUT"
+		(at 99.06 81.28 0)
+		(effects
+			(font
+				(size 1.27 1.27)
+			)
+			(justify left bottom)
+		)
+	)
 	(label "+VE"
 		(at 139.7 111.76 0)
@@
 		)
 		(instances
-			(project "Untitled"
+			(project "schematics"
 				(path "/a2c6df74-bcdc-42fd-aec1-9beaf5725762"
 					(reference "#PWR05")
@@
 		)
 		(instances
-			(project "Untitled"
+			(project "schematics"
 				(path "/a2c6df74-bcdc-42fd-aec1-9beaf5725762"
 					(reference "#PWR09")
@@
 		)
 		(instances
-			(project "Untitled"
+			(project "schematics"
 				(path "/a2c6df74-bcdc-42fd-aec1-9beaf5725762"
 					(reference "J1")
@@
 		)
 		(instances
-			(project "Untitled"
+			(project "schematics"
 				(path "/a2c6df74-bcdc-42fd-aec1-9beaf5725762"
 					(reference "#PWR010")
@@
 		)
 		(instances
-			(project "Untitled"
+			(project "schematics"
 				(path "/a2c6df74-bcdc-42fd-aec1-9beaf5725762"
 					(reference "J5")
@@
 		)
 		(instances
-			(project "Untitled"
+			(project "schematics"
 				(path "/a2c6df74-bcdc-42fd-aec1-9beaf5725762"
 					(reference "#PWR012")
@@
 		)
 		(instances
-			(project "Untitled"
+			(project "schematics"
 				(path "/a2c6df74-bcdc-42fd-aec1-9beaf5725762"
 					(reference "#PWR08")
@@
 		)
 		(instances
-			(project "Untitled"
+			(project "schematics"
 				(path "/a2c6df74-bcdc-42fd-aec1-9beaf5725762"
 					(reference "#PWR04")
@@
 		)
 		(instances
-			(project "Untitled"
+			(project "schematics"
 				(path "/a2c6df74-bcdc-42fd-aec1-9beaf5725762"
 					(reference "#PWR06")
@@
 		)
 		(instances
-			(project "Untitled"
+			(project "schematics"
 				(path "/a2c6df74-bcdc-42fd-aec1-9beaf5725762"
 					(reference "#PWR07")
@@
 		)
 		(instances
-			(project "Untitled"
+			(project "schematics"
 				(path "/a2c6df74-bcdc-42fd-aec1-9beaf5725762"
 					(reference "SW2")
@@
 		)
 		(instances
-			(project "Untitled"
+			(project "schematics"
 				(path "/a2c6df74-bcdc-42fd-aec1-9beaf5725762"
 					(reference "#PWR01")
@@
 		)
 		(instances
-			(project "Untitled"
+			(project "schematics"
 				(path "/a2c6df74-bcdc-42fd-aec1-9beaf5725762"
 					(reference "#PWR013")
@@
 		)
 		(instances
-			(project "Untitled"
+			(project "schematics"
 				(path "/a2c6df74-bcdc-42fd-aec1-9beaf5725762"
 					(reference "#PWR02")
@@
 		)
 		(instances
-			(project "Untitled"
+			(project "schematics"
 				(path "/a2c6df74-bcdc-42fd-aec1-9beaf5725762"
 					(reference "#PWR014")
@@
 		)
 		(instances
-			(project "Untitled"
+			(project "schematics"
 				(path "/a2c6df74-bcdc-42fd-aec1-9beaf5725762"
 					(reference "J4")
@@
 		)
 		(instances
-			(project "Untitled"
+			(project "schematics"
 				(path "/a2c6df74-bcdc-42fd-aec1-9beaf5725762"
 					(reference "#PWR03")
@@
 		)
 		(instances
-			(project "Untitled"
+			(project "schematics"
 				(path "/a2c6df74-bcdc-42fd-aec1-9beaf5725762"
 					(reference "U1")
@@
 		)
 		(instances
-			(project "Untitled"
+			(project "schematics"
 				(path "/a2c6df74-bcdc-42fd-aec1-9beaf5725762"
 					(reference "J2")
@@
 		)
 		(instances
-			(project "Untitled"
+			(project "schematics"
 				(path "/a2c6df74-bcdc-42fd-aec1-9beaf5725762"
 					(reference "#PWR011")
@@
 		)
 		(instances
-			(project "Untitled"
+			(project "schematics"
 				(path "/a2c6df74-bcdc-42fd-aec1-9beaf5725762"
 					(reference "J3")
